File: PCB/TINYPLAY_PCB/TINYPLAY_PCB.kicad_pcb (KiCad board)
At the start: 2 copper layers, 18.5 x 18.5 mm, 18 parts, among them J1 Conn_02x03_Odd_Even, J6 Conn_01x04_Male, J7 Conn_01x04_Male, SW1 SW_SPDT, SW2 SW_Push, SW3 SW_Push, U1 ATtiny5-TS, U2 74HC164

Commit message: Version 2.0
Other:
- board text added: "TINYPLAYv2 Adam Anderson 2022"
Changed lines of the file:
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@@
       (psnegative false)
       (psa4output false)
-      (plotreference true)
-      (plotvalue true)
+      (plotreference false)
+      (plotvalue false)
       (plotinvisibletext false)
       (sketchpadsonfab false)
@@
       (outputformat 1)
       (mirror false)
-      (drillshape 1)
+      (drillshape 0)
       (scaleselection 1)
-      (outputdirectory "")
+      (outputdirectory "TINYPLAY_PCB_GRB/")
     )
   )
@@
   (gr_arc (start 81 47.5) (mid 80.292893 47.207107) (end 80 46.5) (layer "Edge.Cuts") (width 0.1))
   (gr_line (start 97.5 47.5) (end 81 47.5) (layer "Edge.Cuts") (width 0.1))
+  (gr_text "TINYPLAYv2\nAdam Anderson\n2022" (at 95.8 38.8 90) (layer "F.SilkS")
+    (effects (font (size 1 1) (thickness 0.2)))
+  )
   (target plus (at 89.2 38.8) (size 5) (width 0.1) (layer "Edge.Cuts"))
   (segment (start 87.4375 45.15) (end 87.053928 45.15) (width 0.25) (layer "F.Cu") (net 1))
